File: Rev000/OpenLoopFullElectrical_000/OpenLoopFullElectrical_000.sch (KiCad schematic (older format))
At the start: 71 parts, among them J101 CONN_01X08, J102 CONN_01X02, J103 CONN_01X08, J104 CONN_01X08, J110 CONN_02X04, J111 CONN_02X04, J112 CONN_02X04, J113 CONN_02X04, J120 CONN_01X02, J121 CONN_01X02, J122 CONN_01X02, J123 CONN_01X02, J130 CONN_01X02, J132 CONN_01X02, J134 CONN_01X02, J136 CONN_02X12, J137 CONN_02X04, U110 LM7824CT, U111 LM7824CT, U112 LM7824CT, U113 LM7824CT, U120 LM7824CT, U121 LM7824CT, U122 LM7824CT, U123 LM7824CT, U130 LM7824CT, U131 LM2931Z-5.0, U132 LM7824CT, U133 LM2931Z-5.0, U134 LM7824CT, U135 LM2931Z-5.0, U136 LM7824CT, U137 LM2931Z-5.0

Commit message: Created root schematic which contains all other schematic pages (it's kind of annoying, but that's how KiCad does it...)
Parts:
- removed C101, C102, C103, C104, C105: 10u, symbol C
- removed C110, C112, C114, C116, C120, C122, C124, C125, C130, C134, C138, C142: 0.33uF, symbol C
- removed C111, C113, C115, C117, C121, C123, C125, C126, C131, C135, C139, C143: 0.1uF, symbol C
- removed C132, C136, C140, C144: 0.47uF, symbol C
- removed C133, C137, C141, C145: 47uF, symbol C
- removed J101, J103, J104: CONN_01X08, symbol CONN_01X08
- removed J102, J120, J121, J122, J123, J130, J132, J134: CONN_01X02, symbol CONN_01X02
- removed J110, J111, J112, J113, J137: CONN_02X04, symbol CONN_02X04
- removed J136: CONN_02X12, symbol CONN_02X12
- removed Q?: MOSFET_N, symbol MOSFET_N
- removed U110, U111, U112, U113, U120, U121, U122, U123, U130, U132, U134, U136: LM7824CT, TO-220, symbol LM7824CT
- removed U131, U133, U135, U137: LM2931Z-5.0, TO92-123, symbol LM2931Z-5.0
Connections:
- net labels removed: +36V, 24V0_TO_CPU_LR, 24V0_TO_IMU, 24V0_TO_MPYE1, 24V0_TO_MPYE2, 24V0_TO_MUX_LR, 24V0_TO_NAP, 24V0_TO_RB_LR1, 24V0_TO_RB_LR2, 24V0_TO_SOL1, 24V0_TO_SOL2, 24V0_TO_SOL3, 24V0_TO_SOL4, 36V0_BATT, 5V0_TO_CPU, 5V0_TO_MUX, 5V0_TO_RB1, 5V0_TO_RB2, GND
- wire segments 254 -> 0
Other:
- note added: "KiCad is annoying about using multiple pages - in order to do it,\nwe have to have this root schematic file which contains hierarchical\npages which represent each schematic page.\n\nTo access schematics, you need to open them through this sheet.\nIf you open them directly from KiCad, none of the schematic symbols\nwill populate correctly. Just double click on a page to enter it, and when\nyou’re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"
- note added: "Table of Contents"
- note removed: "Battery"
- note removed: "Battery connection\n\n36V and GND references originate here"
- note removed: "Bypass caps - locate close to U101\n"
- note removed: "Connector to BBB for enabling battery"
- note removed: "MOSFET for controlling battery input"
- note removed: "Power to Back Board\n"
- note removed: "Power to CPU\n"
- note removed: "Power to Front Board\n"
- note removed: "Power to Front/Back Boards"
- note removed: "Power to IMU"
- note removed: "Power to Linear Proportional\nControl Valves (MPYEs)"
- note removed: "Power to MUX/DEMUX, OMRON, TCC, and SHARP\n"
- note removed: "Power to NAP\n"
- note removed: "Power to Relay Boards\n"
- note removed: "Power to Solenoids\n"
